File: 8bitWave Faceplate/8bitWave Faceplate.sch (KiCad schematic (older format))
At the start: 44 parts, among them IC1 0.96_I2C_OLED, J1 I2C_VOL, J3 EXTENSION, M1 Mounting, M2 Mounting, M3 Mounting, M4 Mounting, U1 74HC595_ALT

Commit message: Finishing touches
Parts:
- J1: symbol Conn_01x03 -> I2C_VOLTAGE
- J3: symbol Conn_01x07 -> Extension
- gave numbers to parts that had none: 17
Connections:
- net +3V3 is gone; now on net VCC: J1.1 (Pin_1)
Other:
- note added: "Over-engineered by design, but it's all in a days fun so extended it to include some SMD\nblinkenlights. The only needed components is just the OLED display."
Changed lines of the file:
@@
 LIBS:audio_jack
 LIBS:74hc595_alt
+LIBS:i2c_voltage
+LIBS:extension
 LIBS:8bitWave Faceplate-cache
 EELAYER 25 0
@@
 encoding utf-8
 Sheet 1 1
-Title ""
+Title "8BIT WAVE Faceplate"
 Date ""
-Rev ""
+Rev "A"
 Comp ""
 Comment1 ""
@@
 	-1   0    0    -1
 $EndComp
-$Comp
-L +3.3V #PWR01
-U 1 1 5E3B7508
-P 3825 1650
-F 0 "#PWR01" H 3825 1500 50  0001 C CNN
-F 1 "+3.3V" H 3825 1790 50  0000 C CNN
-F 2 "" H 3825 1650 50  0001 C CNN
-F 3 "" H 3825 1650 50  0001 C CNN
-	1    3825 1650
-	-1   0    0    -1
-$EndComp
 Text Label 7275 1700 0    60   ~ 0
 SCL
@@
 	5600 1850 7150 1850
 $Comp
-L Conn_01x07 J3
+L Extension J3
 U 1 1 5E3D299E
 P 4650 1775
@@
 $EndComp
 $Comp
-L GND #PWR02
+L GND #PWR01
 U 1 1 5E3D3470
 P 4925 2150
-F 0 "#PWR02" H 4925 1900 50  0001 C CNN
+F 0 "#PWR01" H 4925 1900 50  0001 C CNN
 F 1 "GND" H 4925 2000 50  0000 C CNN
 F 2 "" H 4925 2150 50  0001 C CNN
@@
 SHIFT_DATA
 $Comp
-L Conn_01x03 J1
+L I2C_VOLTAGE J1
 U 1 1 5E3E91C2
 P 3550 1825
@@
 $EndComp
 Wire Wire Line
-	3825 1650 3825 1725
-Wire Wire Line
 	3825 1725 3750 1725
 $Comp
-L +5V #PWR03
+L +5V #PWR02
 U 1 1 5E3EA726
 P 4125 1850
-F 0 "#PWR03" H 4125 1700 50  0001 C CNN
+F 0 "#PWR02" H 4125 1700 50  0001 C CNN
 F 1 "+5V" H 4125 1990 50  0000 C CNN
 F 2 "" H 4125 1850 50  0001 C CNN
@@
 $EndComp
 $Comp
-L GND #PWR04
+L GND #PWR03
 U 1 1 5E3ED47A
 P 5750 1550
-F 0 "#PWR04" H 5750 1300 50  0001 C CNN
+F 0 "#PWR03" H 5750 1300 50  0001 C CNN
 F 1 "GND" H 5750 1400 50  0000 C CNN
 F 2 "" H 5750 1550 50  0001 C CNN
@@
 	3750 1925 4125 1925
 $Comp
-L VCC #PWR05
+L VCC #PWR04
 U 1 1 5E3EF557
 P 3975 1750
-F 0 "#PWR05" H 3975 1600 50  0001 C CNN
+F 0 "#PWR04" H 3975 1600 50  0001 C CNN
 F 1 "VCC" H 3975 1900 50  0000 C CNN
 F 2 "" H 3975 1750 50  0001 C CNN
@@
 	8825 1700 8825 1800
 $Comp
-L GND #PWR06
+L GND #PWR05
 U 1 1 5E3EF7B8
 P 8825 1800
-F 0 "#PWR06" H 8825 1550 50  0001 C CNN
+F 0 "#PWR05" H 8825 1550 50  0001 C CNN
 F 1 "GND" H 8825 1650 50  0000 C CNN
 F 2 "" H 8825 1800 50  0001 C CNN
@@
 $EndComp
 $Comp
-L VCC #PWR07
+L VCC #PWR06
 U 1 1 5E3EF86D
 P 8400 1700
-F 0 "#PWR07" H 8400 1550 50  0001 C CNN
+F 0 "#PWR06" H 8400 1550 50  0001 C CNN
 F 1 "VCC" H 8400 1850 50  0000 C CNN
 F 2 "" H 8400 1700 50  0001 C CNN
@@
 	5600 1675 5600 2075
 $Comp
-L GND #PWR08
+L GND #PWR07
 U 1 1 5E3F40C6
 P 4125 4975
-F 0 "#PWR08" H 4125 4725 50  0001 C CNN
+F 0 "#PWR07" H 4125 4725 50  0001 C CNN
 F 1 "GND" H 4125 4825 50  0000 C CNN
 F 2 "" H 4125 4975 50  0001 C CNN
@@
 $EndComp
 $Comp
-L +5V #PWR09
+L +5V #PWR08
 U 1 1 5E3F43A4
 P 4225 3375
-F 0 "#PWR09" H 4225 3225 50  0001 C CNN
+F 0 "#PWR08" H 4225 3225 50  0001 C CNN
 F 1 "+5V" H 4225 3515 50  0000 C CNN
 F 2 "" H 4225 3375 50  0001 C CNN
@@
 $EndComp
 $Comp
-L +5V #PWR010
+L +5V #PWR09
 U 1 1 5E3F69AA
 P 10375 5625
-F 0 "#PWR010" H 10375 5475 50  0001 C CNN
+F 0 "#PWR09" H 10375 5475 50  0001 C CNN
 F 1 "+5V" H 10375 5765 50  0000 C CNN
 F 2 "" H 10375 5625 50  0001 C CNN
@@
 	10925 6075 10925 6225
 $Comp
-L GND #PWR011
+L GND #PWR010
 U 1 1 5E3F6B5B
 P 10925 6225
-F 0 "#PWR011" H 10925 5975 50  0001 C CNN
+F 0 "#PWR010" H 10925 5975 50  0001 C CNN
 F 1 "GND" H 10925 6075 50  0000 C CNN
 F 2 "" H 10925 6225 50  0001 C CNN
@@
 	2750 3725 2750 4500
 $Comp
-L GND #PWR012
+L GND #PWR011
 U 1 1 5E3F7B9C
 P 2750 4500
-F 0 "#PWR012" H 2750 4250 50  0001 C CNN
+F 0 "#PWR011" H 2750 4250 50  0001 C CNN
 F 1 "GND" H 2750 4350 50  0000 C CNN
 F 2 "" H 2750 4500 50  0001 C CNN
@@
 Connection ~ 2750 3825
 $Comp
-L GND #PWR?
+L GND #PWR012
 U 1 1 5E3F8B26
 P 4125 7100
-F 0 "#PWR?" H 4125 6850 50  0001 C CNN
+F 0 "#PWR012" H 4125 6850 50  0001 C CNN
 F 1 "GND" H 4125 6950 50  0000 C CNN
 F 2 "" H 4125 7100 50  0001 C CNN
@@
 $EndComp
 $Comp
-L 74HC595_ALT U?
+L 74HC595_ALT U2
 U 1 1 5E3F8B2C
 P 4175 6300
-F 0 "U?" H 4525 6900 50  0000 C CNN
+F 0 "U2" H 4525 6900 50  0000 C CNN
 F 1 "74HC595_ALT" V 4175 6300 50  0000 C CNN
 F 2 "SMD_Packages:SO-16-N" H 4175 6300 50  0001 C CNN
@@
 $EndComp
 $Comp
-L +5V #PWR?
+L +5V #PWR013
 U 1 1 5E3F8B32
 P 4225 5500
-F 0 "#PWR?" H 4225 5350 50  0001 C CNN
+F 0 "#PWR013" H 4225 5350 50  0001 C CNN
 F 1 "+5V" H 4225 5640 50  0000 C CNN
 F 2 "" H 4225 5500 50  0001 C CNN
@@
 NoConn ~ 4875 6750
 $Comp
-L R R?
+L R R9
 U 1 1 5E3F8B4A
 P 3250 5850
-F 0 "R?" V 3330 5850 50  0001 C CNN
+F 0 "R9" V 3330 5850 50  0001 C CNN
 F 1 "330" V 3250 5850 50  0000 C CNN
 F 2 "Resistors_SMD:R_0805_HandSoldering" V 3180 5850 50  0001 C CNN
@@
 	3400 5850 3475 5850
 $Comp
-L LED_Small D?
+L LED_Small D9
 U 1 1 5E3F8B51
 P 2925 5850
-F 0 "D?" H 2975 5900 50  0000 L CNN
+F 0 "D9" H 2975 5900 50  0000 L CNN
 F 1 "RED" H 2750 5750 50  0001 L CNN
 F 2 "LEDs:LED_0805_HandSoldering" V 2925 5850 50  0001 C CNN
@@
 	2825 5850 2750 5850
 $Comp
-L R R?
+L R R10
 U 1 1 5E3F8B59
 P 3250 5950
-F 0 "R?" V 3330 5950 50  0001 C CNN
+F 0 "R10" V 3330 5950 50  0001 C CNN
 F 1 "330" V 3250 5950 50  0000 C CNN
 F 2 "Resistors_SMD:R_0805_HandSoldering" V 3180 5950 50  0001 C CNN
@@
 	3400 5950 3475 5950
 $Comp
-L LED_Small D?
+L LED_Small D10
 U 1 1 5E3F8B60
 P 2925 5950
-F 0 "D?" H 2975 6000 50  0000 L CNN
+F 0 "D10" H 2975 6000 50  0000 L CNN
 F 1 "RED" H 2750 5850 50  0001 L CNN
 F 2 "LEDs:LED_0805_HandSoldering" V 2925 5950 50  0001 C CNN
@@
 	2825 5950 2750 5950
 $Comp
-L R R?
+L R R11
 U 1 1 5E3F8B68
 P 3250 6050
-F 0 "R?" V 3330 6050 50  0001 C CNN
+F 0 "R11" V 3330 6050 50  0001 C CNN
 F 1 "330" V 3250 6050 50  0000 C CNN
 F 2 "Resistors_SMD:R_0805_HandSoldering" V 3180 6050 50  0001 C CNN
@@
 	3400 6050 3475 6050
 $Comp
-L LED_Small D?
+L LED_Small D11
 U 1 1 5E3F8B6F
 P 2925 6050
-F 0 "D?" H 2975 6100 50  0000 L CNN
+F 0 "D11" H 2975 6100 50  0000 L CNN
 F 1 "RED" H 2750 5950 50  0001 L CNN
 F 2 "LEDs:LED_0805_HandSoldering" V 2925 6050 50  0001 C CNN
@@
 	2825 6050 2750 6050
 $Comp
-L R R?
+L R R12
 U 1 1 5E3F8B77
 P 3250 6150
-F 0 "R?" V 3330 6150 50  0001 C CNN
+F 0 "R12" V 3330 6150 50  0001 C CNN
 F 1 "330" V 3250 6150 50  0000 C CNN
 F 2 "Resistors_SMD:R_0805_HandSoldering" V 3180 6150 50  0001 C CNN
@@
 	3400 6150 3475 6150
 $Comp
-L LED_Small D?
+L LED_Small D12
 U 1 1 5E3F8B7E
 P 2925 6150
-F 0 "D?" H 2975 6200 50  0000 L CNN
+F 0 "D12" H 2975 6200 50  0000 L CNN
 F 1 "RED" H 2750 6050 50  0001 L CNN
 F 2 "LEDs:LED_0805_HandSoldering" V 2925 6150 50  0001 C CNN
@@
 	2825 6150 2750 6150
 $Comp
-L R R?
+L R R13
 U 1 1 5E3F8B86
 P 3250 6250
-F 0 "R?" V 3330 6250 50  0001 C CNN
+F 0 "R13" V 3330 6250 50  0001 C CNN
 F 1 "330" V 3250 6250 50  0000 C CNN
 F 2 "Resistors_SMD:R_0805_HandSoldering" V 3180 6250 50  0001 C CNN
@@
 	3400 6250 3475 6250
 $Comp
-L LED_Small D?
+L LED_Small D13
 U 1 1 5E3F8B8D
 P 2925 6250
-F 0 "D?" H 2975 6300 50  0000 L CNN
+F 0 "D13" H 2975 6300 50  0000 L CNN
 F 1 "RED" H 2750 6150 50  0001 L CNN
 F 2 "LEDs:LED_0805_HandSoldering" V 2925 6250 50  0001 C CNN
@@
 	2825 6250 2750 6250
 $Comp
-L R R?
+L R R14
 U 1 1 5E3F8B95
 P 3250 6350
-F 0 "R?" V 3330 6350 50  0001 C CNN
+F 0 "R14" V 3330 6350 50  0001 C CNN
 F 1 "330" V 3250 6350 50  0000 C CNN
 F 2 "Resistors_SMD:R_0805_HandSoldering" V 3180 6350 50  0001 C CNN
@@
 	3400 6350 3475 6350
 $Comp
-L LED_Small D?
+L LED_Small D14
 U 1 1 5E3F8B9C
 P 2925 6350
-F 0 "D?" H 2975 6400 50  0000 L CNN
+F 0 "D14" H 2975 6400 50  0000 L CNN
 F 1 "RED" H 2750 6250 50  0001 L CNN
 F 2 "LEDs:LED_0805_HandSoldering" V 2925 6350 50  0001 C CNN
@@
 	2825 6350 2750 6350
 $Comp
-L R R?
+L R R15
 U 1 1 5E3F8BA4
 P 3250 6450
-F 0 "R?" V 3330 6450 50  0001 C CNN
+F 0 "R15" V 3330 6450 50  0001 C CNN
 F 1 "330" V 3250 6450 50  0000 C CNN
 F 2 "Resistors_SMD:R_0805_HandSoldering" V 3180 6450 50  0001 C CNN
@@
 	3400 6450 3475 6450
 $Comp
-L LED_Small D?
+L LED_Small D15
 U 1 1 5E3F8BAB
 P 2925 6450
-F 0 "D?" H 2975 6500 50  0000 L CNN
+F 0 "D15" H 2975 6500 50  0000 L CNN
 F 1 "RED" H 2750 6350 50  0001 L CNN
 F 2 "LEDs:LED_0805_HandSoldering" V 2925 6450 50  0001 C CNN
@@
 	2825 6450 2750 6450
 $Comp
-L R R?
+L R R16
 U 1 1 5E3F8BB3
 P 3250 6550
-F 0 "R?" V 3330 6550 50  0001 C CNN
+F 0 "R16" V 3330 6550 50  0001 C CNN
 F 1 "330" V 3250 6550 50  0000 C CNN
 F 2 "Resistors_SMD:R_0805_HandSoldering" V 3180 6550 50  0001 C CNN
@@
 	3400 6550 3475 6550
 $Comp
-L LED_Small D?
+L LED_Small D16
 U 1 1 5E3F8BBA
 P 2925 6550
-F 0 "D?" H 2975 6600 50  0000 L CNN
+F 0 "D16" H 2975 6600 50  0000 L CNN
 F 1 "RED" H 2750 6450 50  0001 L CNN
 F 2 "LEDs:LED_0805_HandSoldering" V 2925 6550 50  0001 C CNN
@@
 	2750 5850 2750 6625
 $Comp
-L GND #PWR?
+L GND #PWR014
 U 1 1 5E3F8BC3
 P 2750 6625
-F 0 "#PWR?" H 2750 6375 50  0001 C CNN
+F 0 "#PWR014" H 2750 6375 50  0001 C CNN
 F 1 "GND" H 2750 6475 50  0000 C CNN
 F 2 "" H 2750 6625 50  0001 C CNN
@@
 Wire Wire Line
 	4950 5850 4875 5850
+Wire Wire Line
+	3825 1725 3825 1825
+Connection ~ 3825 1825
+Text Notes 7000 6750 0    60   ~ 0
+Over-engineered by design, but it's all in a days fun so extended it to include some SMD\nblinkenlights. The only needed components is just the OLED display.
 $EndSCHEMATC
