File: 8bitWave Module/8bitWave Module.sch (KiCad schematic (older format))
At the start: 35 parts, among them IC1 0.96_I2C_OLED, IC2 0.91_I2C_OLED, J1 REM, J2 EAR, M1 Mounting, M2 Mounting, M3 Mounting, M4 Mounting, SW1 UP, SW2 DOWN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

Commit message: Layout sketched out
Parts:
- added D1: POWER, LEDs:LED_D5.0mm, symbol LED_Small
- added D2: USER, LEDs:LED_D5.0mm, symbol LED_Small
- added J3: Faceplate, Pin_Headers:Pin_Header_Straight_1x08_Pitch2.54mm, symbol Conn_01x08
- added JP4: BYPASS, Pin_Headers:Pin_Header_Straight_1x02_Pitch2.54mm, symbol Jumper_NO_Small
- added R6, R7: 220, Resistors_THT:R_Axial_DIN0207_L6.3mm_D2.5mm_P10.16mm_Horizontal, symbol R
Connections:
- net +3V3: now also J3.1 (Pin_1)
- net +5V: now also J3.7 (Pin_7)
- net GND: now also D1.1 (K), D2.1 (K), J3.8 (Pin_8), JP4.2; no longer C7.2
- net SCL: now also J3.6 (Pin_6)
- net SDA: now also J3.5 (Pin_5)
- net SOUND: now also JP2.1; no longer JP2.2
- net D8: now reaches A1.11 (D8)
- net D8: now also J3.2 (Pin_2)
- net D2: now reaches A1.5 (D2)
- net D2: now also J3.4 (Pin_4)
- net USER: now reaches A1.6 (D3)
- net USER: now also R7.2
- net D4: now reaches A1.7 (D4)
- net D4: now also J3.3 (Pin_3)
- net POWER: now reaches A1.8 (D5)
- net POWER: now also R6.2
- net at C1.2, R4.2, RV1.2: now also JP2.2; no longer JP2.1
- new net: D1.2 (A), R6.1
- new net: C7.2, JP4.1
- new net: D2.2 (A), R7.1
- no-connect marks 17 -> 12
Other:
- note added: "Noise\n-reduction"
- moved on the sheet: C5, C6, C7

Commit message: Tweaked silkscreen
Parts:
- added JP5: I2C_VOL, Pin_Headers:Pin_Header_Straight_1x03_Pitch2.54mm, symbol Jumper_NC_Dual
- added R8, R9: 4k7, Resistors_THT:R_Axial_DIN0207_L6.3mm_D2.5mm_P10.16mm_Horizontal, symbol R
- A1: value Arduino_Nano_v3.x -> Arduino Nano
- A2: value MicroSD -> MicroSD Card Adapter
- J3: value Faceplate -> EXTENSION; footprint Pin_Headers:Pin_Header_Straight_1x08_Pitch2.54mm -> Pin_Headers:Pin_Header_Straight_1x07_Pitch2.54mm; symbol Conn_01x08 -> Conn_01x07
Connections:
- net +3V3: now also JP5.1; no longer IC1.2 (VCC), IC2.2 (VCC), J3.1 (Pin_1)
- net +5V: now also JP5.3; no longer J3.7 (Pin_7)
- net GND: now also J3.1 (Pin_1), J3.7 (Pin_7); no longer J3.8 (Pin_8)
- net SCL: now also R8.1
- net SDA: now also R9.1
- net SOUND: now also JP3.1; no longer JP3.3
- net at C10.2, C9.1: now also JP3.3; no longer JP3.1
- new net: IC1.2 (VCC), IC2.2 (VCC), JP5.2, R8.2, R9.2
Other:
- note added: "OLEDs usually include\nthese, no need to\ninstall unless needed."
- note added: "OLEDs usually work\nin either position,\nlink pins 1-2 for 3.3v."
- moved on the sheet: IC1, IC2

Commit message: Finishing touches
Parts:
- A1: symbol Arduino_Nano_v3.x -> Arduino_Nano
- JP5: symbol Jumper_NC_Dual -> I2C_VOLTAGE_SELECT
Other:
- note added: "Based on the DigiWavuino, but I wanted to build my own version of it with a lot of\nfeatures no one would ever need - mostly because I wanted to play around with\nvarious things Arduino. There is an option for using either an 128x32 or 128x64 OLED,\ninstall whichever you want and hope that the software supports it - alternatively, use\none of the available faceplates and install the display there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"
Changed lines of the file:
@@
 LIBS:microsd_adapter
 LIBS:audio_jack
+LIBS:arduino_nano
+LIBS:i2c_voltage_select
 LIBS:8bitWave Module-cache
 EELAYER 25 0
@@
 encoding utf-8
 Sheet 1 1
-Title ""
+Title "8BIT WAVE"
 Date ""
-Rev ""
+Rev "A"
 Comp ""
 Comment1 ""
@@
 $EndComp
 $Comp
-L Arduino_Nano_v3.x A1
+L Arduino_Nano A1
 U 1 1 5E3B6403
 P 6700 3550
@@
 $EndComp
 $Comp
-L Jumper_NC_Dual JP5
+L I2C_VOLTAGE_SELECT JP5
 U 1 1 5E3E91C2
 P 6475 1025
@@
 Text Notes 5925 1025 2    60   ~ 0
 OLEDs usually work\nin either position,\nlink pins 1-2 for 3.3v.
+Text Notes 7000 7025 0    60   ~ 0
+Based on the DigiWavuino, but I wanted to build my own version of it with a lot of\nfeatures no one would ever need - mostly because I wanted to play around with\nvarious things Arduino. There is an option for using either an 128x32 or 128x64 OLED,\ninstall whichever you want and hope that the software supports it - alternatively, use\none of the available faceplates and install the display there instead.
 $EndSCHEMATC
