File: 8bitWave Module/8bitWave Module.sch (KiCad schematic (older format))
At the start: 49 parts, among them IC1 0.96_OLED, J1 REM, J2 EAR, J3 EXTENSION, J4 DC IN, J5 LP_FILTER, J6 SPI, J7 EAR_SEL, M1 Mounting, M2 Mounting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

Commit message: Updated module (KiCad 5)
Parts:
- J3: symbol 8bitWave-Module-rescue:Conn_01x07-conn-8bitWave-Module-rescue -> Connector_Generic:Conn_01x07
- J5: symbol 8bitWave-Module-rescue:Conn_02x03_Odd_Even-conn-8bitWave-Module-rescue -> Connector_Generic:Conn_02x03_Odd_Even
- J6: symbol 8bitWave-Module-rescue:Conn_01x03-conn-8bitWave-Module-rescue -> Connector_Generic:Conn_01x03
- J7: symbol 8bitWave-Module-rescue:Conn_02x06_Odd_Even-conn-8bitWave-Module-rescue -> Connector_Generic:Conn_02x06_Odd_Even
- RV2: symbol 8bitWave-Module-rescue:POT-8bitWave-Module-rescue -> Device:R_POT
- SW1, SW2, SW3, SW4, SW5: symbol 8bitWave-Module-rescue:SW_SPST-switches-8bitWave-Module-rescue -> Switch:SW_Push
- U1: symbol 8bitWave-Module-rescue:LM386-linear-8bitWave-Module-rescue -> Amplifier_Audio:LM386
Changed lines of the file:
@@
 $EndComp
 $Comp
-L 8bitWave-Module-rescue:SW_SPST-switches-8bitWave-Module-rescue SW1
+L Switch:SW_Push SW1
 U 1 1 5E3B6481
 P 14100 4650
@@
 $EndComp
 $Comp
-L 8bitWave-Module-rescue:SW_SPST-switches-8bitWave-Module-rescue SW2
+L Switch:SW_Push SW2
 U 1 1 5E3B64CB
 P 14100 5000
@@
 $EndComp
 $Comp
-L 8bitWave-Module-rescue:SW_SPST-switches-8bitWave-Module-rescue SW3
+L Switch:SW_Push SW3
 U 1 1 5E3B64F8
 P 14100 5350
@@
 $EndComp
 $Comp
-L 8bitWave-Module-rescue:SW_SPST-switches-8bitWave-Module-rescue SW4
+L Switch:SW_Push SW4
 U 1 1 5E3B6550
 P 14100 5700
@@
 $EndComp
 $Comp
-L 8bitWave-Module-rescue:SW_SPST-switches-8bitWave-Module-rescue SW5
+L Switch:SW_Push SW5
 U 1 1 5E3B65A5
 P 14100 6050
@@
 $EndComp
 $Comp
-L 8bitWave-Module-rescue:LM386-linear-8bitWave-Module-rescue U1
+L Amplifier_Audio:LM386 U1
 U 1 1 5E3CBAD8
 P 2800 6550
@@
 POWER
 $Comp
-L 8bitWave-Module-rescue:Conn_01x07-conn-8bitWave-Module-rescue J3
+L Connector_Generic:Conn_01x07 J3
 U 1 1 5E3D299E
 P 11975 5700
@@
 Wire Notes Line
 	10675 1400 10675 725
-Text Notes 10600 1175 2    60   ~ 0
+Text Notes 10550 1175 2    60   ~ 0
 OLEDs usually work\nin either position,\nlink pins 1-2 for 3.3v.
-Text Notes 11850 10475 0    60   ~ 0
+Text Notes 11850 10375 0    60   ~ 0
 Based on the DigiWavuino, but I wanted to build my own version of it with a lot of\nfeatures no one would ever need - mostly because I wanted to play around with\nvarious things Arduino. A 128x64 OLED can be mounted directly, but the main goal of\nthe project was to hide most things behind a faceplate instead,
 Wire Wire Line
@@
 PWR_SEL positions 1-2 is used when powering amplifier from\nvia Arduino, or when connecting a 5v supply directly.  Positions\n2-3 is used when powering the entire circuit using a 9-12v DC \nsupply. Unjumpered, the amplifier and the rest of the circuit will\neach need their own power source.
 $Comp
-L 8bitWave-Module-rescue:Conn_02x03_Odd_Even-conn-8bitWave-Module-rescue J5
+L Connector_Generic:Conn_02x03_Odd_Even J5
 U 1 1 5E7A4F51
 P 6175 5700
@@
 LOW-PASS FILTER
 $Comp
-L 8bitWave-Module-rescue:Conn_01x03-conn-8bitWave-Module-rescue J6
+L Connector_Generic:Conn_01x03 J6
 U 1 1 5EC476AB
 P 11975 4950
@@
 AUD_LINE
 $Comp
-L 8bitWave-Module-rescue:Conn_02x06_Odd_Even-conn-8bitWave-Module-rescue J7
+L Connector_Generic:Conn_02x06_Odd_Even J7
 U 1 1 5F81D312
 P 6250 3500
@@
 	13500 775  13500 1400
 $Comp
-L 8bitWave-Module-rescue:POT-8bitWave-Module-rescue RV2
+L Device:R_POT RV2
 U 1 1 5FF950C5
 P 3325 6450
@@
 $EndComp
 Wire Wire Line
-	11600 11075 11600 10875
-Wire Wire Line
 	2800 9275 2800 9425
