File: 8bitWave Faceplate A1/8bitWave Faceplate A1.kicad_pcb (KiCad board)
At the start: 2 copper layers, 99.7 x 64.1 mm, 53 parts, among them IC1 0.96_I2C_OLED, J1 I2C_VOL, J2 SPI, J3 EXTENSION, M1 Mounting, M2 Mounting, M3 Mounting, M4 Mounting, U1 74HC595_ALT, U2 74HC595_ALT

Commit message: Updated faceplate A1 (KiCad 5)
Other:
- rule pad_to_mask_clearance: 0.2 -> 0
