File: 8bitWave Faceplate A1/8bitWave Faceplate A1.sch (KiCad schematic (older format))
At the start: 47 parts, among them IC1 0.96_I2C_OLED, J1 I2C_VOL, J2 SPI, J3 EXTENSION, M1 Mounting, M2 Mounting, M3 Mounting, M4 Mounting, U1 74HC595_ALT, U2 74HC595_ALT

Commit message: Updated faceplate A1 (KiCad 5)
Parts:
- J2: symbol conn:Conn_01x10 -> Connector_Generic:Conn_01x10
Changed lines of the file:
@@
 L mounting:Mounting M1
 U 1 1 5E3B603D
-P 9975 525
-F 0 "M1" H 9975 625 50  0001 C CNN
-F 1 "Mounting" H 9975 450 50  0001 C CNN
-F 2 "mounting:M3" H 9975 525 50  0001 C CNN
-F 3 "" H 9975 525 50  0001 C CNN
-	1    9975 525
+P 10775 550
+F 0 "M1" H 10775 650 50  0001 C CNN
+F 1 "Mounting" H 10775 475 50  0001 C CNN
+F 2 "mounting:M3" H 10775 550 50  0001 C CNN
+F 3 "" H 10775 550 50  0001 C CNN
+	1    10775 550
 	1    0    0    -1
 $EndComp
@@
 	3825 1825 3750 1825
 $Comp
-L conn:Conn_01x10 J2
+L Connector_Generic:Conn_01x10 J2
 U 1 1 5E5F2F04
 P 925 1375
