File: 8bitWave Backplate/8bitWave Backplate.kicad_pcb (KiCad board)
At the start: 2 copper layers, 99.7 x 64.1 mm, 5 parts, among them M1 Mounting, M2 Mounting, M3 Mounting, M4 Mounting

Commit message: Updated backplate (KiCad 5)
Connections:
- M1 pad 1: (no net) -> Net-(M1-Pad1)
- M2 pad 1: (no net) -> Net-(M1-Pad1)
- M3 pad 1: (no net) -> Net-(M1-Pad1)
- M4 pad 1: (no net) -> Net-(M1-Pad1)
Routing:
- added copper zone on B.Cu, net Net-(M1-Pad1)
- removed copper zone on B.Cu, net GND
Other:
- rule pad_to_mask_clearance: 0.2 -> 0
Changed lines of the file:
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@@
-(kicad_pcb (version 20171130) (host pcbnew "(5.1.5)-3")
+(kicad_pcb (version 20171130) (host pcbnew "(5.1.8)-1")
   (general
     (thickness 1.6)
@@
     (pad_size 1.524 1.524)
     (pad_drill 0.762)
-    (pad_to_mask_clearance 0.2)
+    (pad_to_mask_clearance 0)
     (aux_axis_origin 0 0)
     (visible_elements 7FFFFFFF)
@@
   )
   (net 0 "")
-  (net 1 GND)
+  (net 1 "Net-(M1-Pad1)")
   (net_class Default "This is the default net class."
     (clearance 0.2)
@@
     (uvia_dia 0.3)
     (uvia_drill 0.1)
+    (add_net "Net-(M1-Pad1)")
   )
   (module mounting:M3 (layer F.Cu)
@@
     (fp_circle (center 0 0) (end 2.6 0) (layer F.CrtYd) (width 0.05))
     (fp_circle (center 0 0) (end 0 -2.286) (layer F.SilkS) (width 0.12))
-    (pad 1 thru_hole circle (at 0 0) (size 5 5) (drill 3.048) (layers *.Cu *.Mask))
+    (pad 1 thru_hole circle (at 0 0) (size 5 5) (drill 3.048) (layers *.Cu *.Mask)
+      (net 1 "Net-(M1-Pad1)"))
   )
   (module mounting:M3 (layer F.Cu)
@@
     (fp_circle (center 0 0) (end 2.6 0) (layer F.CrtYd) (width 0.05))
     (fp_circle (center 0 0) (end 0 -2.286) (layer F.SilkS) (width 0.12))
-    (pad 1 thru_hole circle (at 0 0) (size 5 5) (drill 3.048) (layers *.Cu *.Mask))
+    (pad 1 thru_hole circle (at 0 0) (size 5 5) (drill 3.048) (layers *.Cu *.Mask)
+      (net 1 "Net-(M1-Pad1)"))
   )
   (module mounting:M3 (layer F.Cu)
@@
     (fp_circle (center 0 0) (end 2.6 0) (layer F.CrtYd) (width 0.05))
     (fp_circle (center 0 0) (end 0 -2.286) (layer F.SilkS) (width 0.12))
-    (pad 1 thru_hole circle (at 0 0) (size 5 5) (drill 3.048) (layers *.Cu *.Mask))
+    (pad 1 thru_hole circle (at 0 0) (size 5 5) (drill 3.048) (layers *.Cu *.Mask)
+      (net 1 "Net-(M1-Pad1)"))
   )
   (module mounting:M3 (layer F.Cu)
@@
     (fp_circle (center 0 0) (end 2.6 0) (layer F.CrtYd) (width 0.05))
     (fp_circle (center 0 0) (end 0 -2.286) (layer F.SilkS) (width 0.12))
-    (pad 1 thru_hole circle (at 0 0) (size 5 5) (drill 3.048) (layers *.Cu *.Mask))
+    (pad 1 thru_hole circle (at 0 0) (size 5 5) (drill 3.048) (layers *.Cu *.Mask)
+      (net 1 "Net-(M1-Pad1)"))
   )
   (module icons:logo locked (layer F.Cu)
@@
     (fp_line (start -7.62 3.556) (end -4.572 -1.524) (layer F.SilkS) (width 0.15))
     (fp_line (start 6.096 1.016) (end 7.62 -1.524) (layer F.SilkS) (width 0.15))
+    (fp_line (start -7.62 3.556) (end -2.032 3.556) (layer F.SilkS) (width 0.15))
+    (fp_line (start 7.62 -1.524) (end -4.572 -1.524) (layer F.SilkS) (width 0.15))
     (fp_text user WAVE (at 1.524 2.54) (layer F.SilkS)
       (effects (font (size 2 2) (thickness 0.15) italic))
     )
-    (fp_line (start -7.62 3.556) (end -2.032 3.556) (layer F.SilkS) (width 0.15))
-    (fp_line (start 7.62 -1.524) (end -4.572 -1.524) (layer F.SilkS) (width 0.15))
     (fp_text user 8BIT (at -1.524 0) (layer F.SilkS)
       (effects (font (size 2 2) (thickness 0.15) italic))
@@
   (gr_line (start 71.755 142.24) (end 168.91 142.24) (angle 90) (layer Edge.Cuts) (width 0.15))
   (gr_arc (start 71.755 140.97) (end 71.755 142.24) (angle 90) (layer Edge.Cuts) (width 0.15))
-  (zone (net 1) (net_name GND) (layer B.Cu) (hatch edge 0.508)
+  (zone (net 1) (net_name "Net-(M1-Pad1)") (layer B.Cu) (hatch edge 0.508)
     (connect_pads (clearance 0.508))
     (min_thickness 0.254)
